Commit message: odometery works

File: urdf/base.xacro (robot description, xacro)
@@ -11,5 +11,5 @@
     <!-- Chassis dimensions -->
     <xacro:property name="chassis_mass" value="1.0" /> <!-- arbitrary value for base mass -->
-    <xacro:property name="chassis_length" value="0.45" />
+    <xacro:property name="chassis_length" value="0.40" />
     <xacro:property name="chassis_width" value="0.2" />
     <xacro:property name="chassis_height" value="0.06" />
@@ -29,8 +29,8 @@
     <xacro:property name="right_y_reflect" value="-1" />
     <!-- INCLUDES -->
-    <xacro:include filename="$(find zinger_description)/urdf/materials.xacro" />
-    <xacro:include filename="$(find zinger_description)/urdf/macros.xacro" />
+    <xacro:include filename="$(find omni_bot2)/urdf/materials.xacro" />
+    <xacro:include filename="$(find omni_bot2)/urdf/macros.xacro" />
     <xacro:if value="$(arg is_simulation)">
-    <xacro:include filename="$(find zinger_description)/urdf/gazebo.xacro" />
+    <xacro:include filename="$(find omni_bot2)/urdf/gazebo.xacro" />
     </xacro:if>
     <!-- MODEL -->
@@ -212,5 +212,5 @@
     <!-- LIDAR -->
     <xacro:sensor_lidar
-        name="rplidar_front"
+        name="scanner_link"
         parent_link="chassis_link"
         chassis_top_relative_height="${0.5 * chassis_height}" />

File: urdf/macros.xacro (robot description, xacro)
@@ -213,8 +213,8 @@
         <joint name="joint_body_to_sensor_lidar_${name}" type="fixed">
             <parent link="${parent_link}"/>
-            <child link="link_sensor_lidar_${name}"/>
+            <child link="scanner_link"/>
             <origin rpy="0 0 0" xyz="${collision_x_offset} ${collision_y_offset} ${collision_z_offset}"/>
         </joint>
-        <link name="link_sensor_lidar_${name}">
+        <link name="scanner_link">
             <visual>
                 <origin rpy="0 0 0" xyz="0.0 0 ${0.5 * length_z}"/>

Commit message: update params file

File: urdf/base.xacro (robot description, xacro)
@@ -214,5 +214,5 @@
         name="scanner_link"
         parent_link="chassis_link"
-        chassis_top_relative_height="${0.5 * chassis_height}" />
+        chassis_top_relative_height="0.1" />
     <!-- Bump -->
     <!-- Sonar -->

File: urdf/macros.xacro (robot description, xacro)
@@ -218,5 +218,5 @@
         <link name="scanner_link">
             <visual>
-                <origin rpy="0 0 0" xyz="0.0 0 ${0.5 * length_z}"/>
+                <origin rpy="0 0 0" xyz="0.0 0 {0.5 * length_z}"/>
                 <geometry>
                     <box size="${length_x} ${length_y} ${length_z}"/>

Commit message: urdf changes

File: urdf/base.xacro (robot description, xacro)
@@ -21,6 +21,6 @@
     <!-- Wheel dimensions -->
     <xacro:property name="wheel_mass" value="0.2" />
-    <xacro:property name="wheel_radius" value="0.04" />
-    <xacro:property name="wheel_width" value="0.05" />
+    <xacro:property name="wheel_radius" value="0.05" />
+    <xacro:property name="wheel_width" value="0.04" />
     <!-- -->
     <xacro:property name="front_x_reflect" value="1" />
@@ -207,5 +207,5 @@
     <!-- Sensors -->
     <!-- IMU -->
-    <xacro:sensor_imu name="imu_center" parent_link="chassis_link">
+    <xacro:sensor_imu name="imu" parent_link="chassis_link">
         <origin rpy="0 0 0" xyz="0.0 0.0 0.0"/>
     </xacro:sensor_imu>
@@ -214,6 +214,15 @@
         name="scanner_link"
         parent_link="chassis_link"
-        chassis_top_relative_height="0.1" />
-    <!-- Bump -->
+        chassis_top_relative_height="0.3" />
+    <!-- front camera -->
+    <xacro:camera
+        name="front_camera_link"
+        parent_link="chassis_link"
+        chassis_top_relative_height="0.3" />
+        <!-- rear camera -->
+    <xacro:camera
+        name="rear_camera_link"
+        parent_link="chassis_link"
+        chassis_top_relative_height="0.3" />
     <!-- Sonar -->
     <!-- IR -->

File: urdf/macros.xacro (robot description, xacro)
@@ -171,10 +171,10 @@
         <xacro:property name="collision_y_offset" value="0.005" />
         <xacro:property name="collision_z_offset" value="${0.5 * length_z}" />
-        <joint name="joint_body_to_sensor_imu_${name}" type="fixed">
+        <joint name="joint_imu_${name}" type="fixed">
             <xacro:insert_block name="origin"/>
             <parent link="${parent_link}"/>
-            <child link="link_sensor_imu_${name}"/>
-        </joint>
-        <link name="link_sensor_imu_${name}">
+            <child link="link_${name}"/>
+        </joint>
+        <link name="link_${name}">
             <visual>
                 <origin xyz="${collision_x_offset} ${collision_y_offset} ${collision_z_offset}"/>
@@ -214,15 +214,16 @@
             <parent link="${parent_link}"/>
             <child link="scanner_link"/>
-            <origin rpy="0 0 0" xyz="${collision_x_offset} ${collision_y_offset} ${collision_z_offset}"/>
+            <origin rpy="0 0 0" xyz="0.14 0 ${chassis_top_relative_height}"/>
         </joint>
         <link name="scanner_link">
             <visual>
-                <origin rpy="0 0 0" xyz="0.0 0 {0.5 * length_z}"/>
-                <geometry>
-                    <box size="${length_x} ${length_y} ${length_z}"/>
-                </geometry>
-            </visual>
-            <collision>
-                <origin rpy="0 0 0" xyz="0.0 0 ${0.5 * length_z}"/>
+                <origin rpy="0 0 0" xyz="0.0 0 0"/>
+                <geometry>
+                    <box size="${length_x} ${length_y} ${length_z}"/>
+                </geometry>
+                <material name="blue"/>
+            </visual>
+            <collision>
+                <origin rpy="0 0 0" xyz="0.0 0 0"/>
                 <geometry>
                     <box size="${length_x} ${length_y} ${length_z}"/>
@@ -231,5 +232,5 @@
             <inertial>
                 <mass value="${mass}" />
-                <origin rpy="0 0 0" xyz="0.0 0 ${0.5 * length_z}"/>
+                <origin rpy="0 0 0" xyz="0.0 0 0"/>
                 <inertia
                     ixx="${(1/12) * mass * (length_y*length_y + length_z*length_z)}"
@@ -242,5 +243,45 @@
         </link>
     </xacro:macro>
-    <!-- Bump sensor -->
+    <!-- camera -->
+    <xacro:macro name="camera" params="name parent_link chassis_top_relative_height">
+        <xacro:property name="mass"     value="0.17"/>
+        <xacro:property name="length_x" value="0.01" />
+        <xacro:property name="length_y" value="0.01" />
+        <xacro:property name="length_z" value="0.01" />
+        <xacro:property name="collision_x_offset" value="-0.07" />
+        <xacro:property name="collision_y_offset" value="-0.2" />
+        <xacro:property name="collision_z_offset" value="${chassis_top_relative_height}" />
+        <joint name="joint_${name}" type="fixed">
+            <parent link="${parent_link}"/>
+            <child link="${name}"/>
+            <origin rpy="0 0 0" xyz="${collision_x_offset} ${collision_y_offset} ${collision_z_offset}"/>
+        </joint>
+        <link name="${name}">
+            <visual>
+                <origin rpy="0 0 0" xyz="0.0 0 0"/>
+                <geometry>
+                    <box size="${length_x} ${length_y} ${length_z}"/>
+                </geometry>
+                <material name="silver"/>
+            </visual>
+            <collision>
+                <origin rpy="0 0 0" xyz="0.0 0 0"/>
+                <geometry>
+                    <box size="${length_x} ${length_y} ${length_z}"/>
+                </geometry>
+            </collision>
+            <inertial>
+                <mass value="${mass}" />
+                <origin rpy="0 0 0" xyz="0.0 0 ${0.5 * length_z}"/>
+                <inertia
+                    ixx="${(1/12) * mass * (length_y*length_y + length_z*length_z)}"
+                    ixy="0.0"
+                    ixz="0.0"
+                    iyy="${(1/12) * mass * (length_x*length_x + length_z*length_z)}"
+                    iyz="0.0"
+                    izz="${(1/12) * mass * (length_x*length_x + length_y*length_y)}" />
+            </inertial>
+        </link>
+    </xacro:macro>
     <!-- Sonar sensor -->
     <!-- IR sensor -->
