Commit message: simple_base

File: urdf/robbie.urdf.xacro (robot description, xacro)
@@ -4,4 +4,5 @@
   <xacro:arg name="add_plug" default="false" />
   <xacro:arg name="use_mesh" default="true" />
+  <xacro:property name="M_PI" value="3.1415926535897931" />
   <xacro:include filename="$(find omni_bot2)/urdf/hardware.xacro" />
   <xacro:include filename="$(find omni_bot2)/urdf/materials.xacro" />
@@ -12,5 +13,5 @@
    <visual>
       <geometry>
-        <mesh filename="package://omni_bot2/mesh/base.stl" scale="${M_SCALE} ${M_SCALE} ${M_SCALE}"/>
+        <mesh filename="package://omni_bot2/mesh/omni_v2_base.stl" scale="${M_SCALE} ${M_SCALE} ${M_SCALE}"/>
       </geometry>
          <xacro:yellow2/>
@@ -20,5 +21,5 @@
         <origin xyz="0 0 0" rpy="0 0 0" />
         <geometry>
-          <mesh filename="package://omni_bot2/mesh/base.stl" scale="${M_SCALE} ${M_SCALE} ${M_SCALE}"/>
+          <mesh filename="package://omni_bot2/mesh/omni_v2_base.stl" scale="${M_SCALE} ${M_SCALE} ${M_SCALE}"/>
           </geometry>
       </collision>
@@ -27,7 +28,7 @@
    <visual>
       <geometry>
-        <mesh filename="package://omni_bot/mesh/X4.stl" scale="${M_SCALE} ${M_SCALE} ${M_SCALE}"/>
+        <mesh filename="package://omni_bot2/mesh/X4.stl" scale="${M_SCALE} ${M_SCALE} ${M_SCALE}"/>
       </geometry>
-         <xacro:black/>
+         <xacro:grey2/>
       <origin rpy="0 0 0" xyz="0 -0 0"/>
     </visual>
@@ -36,4 +37,34 @@
         <geometry>
           <mesh filename="package://omni_bot2/mesh/X4.stl" scale="${M_SCALE} ${M_SCALE} ${M_SCALE}"/>
+          </geometry>
+      </collision>
+  </link>
+  <link name="rear_camera_link" >
+   <visual>
+      <geometry>
+        <mesh filename="package://omni_bot2/mesh/d435.stl" scale="${M_SCALE} ${M_SCALE} ${M_SCALE}"/>
+      </geometry>
+         <xacro:grey1/>
+      <origin rpy="${M_PI/2} 0 -${M_PI/2}" xyz="0 -0 0"/>
+    </visual>
+   <collision>
+        <origin xyz="0 0 0" rpy="${M_PI/2} 0 ${M_PI/2}" />
+        <geometry>
+          <mesh filename="package://omni_bot2/mesh/d435.stl" scale="${M_SCALE} ${M_SCALE} ${M_SCALE}"/>
+          </geometry>
+      </collision>
+  </link>
+  <link name="front_camera_link" >
+   <visual>
+      <geometry>
+        <mesh filename="package://omni_bot2/mesh/d435.stl" scale="${M_SCALE} ${M_SCALE} ${M_SCALE}"/>
+      </geometry>
+         <xacro:grey1/>
+      <origin rpy="1.57 0 1.57" xyz="0 -0 0"/>
+    </visual>
+   <collision>
+        <origin xyz="0 0 0" rpy="1.57 0 1.57" />
+        <geometry>
+          <mesh filename="package://omni_bot2/mesh/d435.stl" scale="${M_SCALE} ${M_SCALE} ${M_SCALE}"/>
           </geometry>
       </collision>
@@ -47,5 +78,15 @@
     	<parent link="base_link" />
     	<child link="scanner_link" />
-    	<origin xyz="0.18 0 0.31" rpy="0 0 0" />
+    	<origin xyz="0.15 0 0.32" rpy="0 0 0" />
+	</joint>
+<joint name="front_camera_link" type="fixed">
+    	<parent link="base_link" />
+    	<child link="front_camera_link" />
+    	<origin xyz="0.0 0 0.35" rpy="0 0 0" />
+	</joint>
+<joint name="rear_camera_link" type="fixed">
+    	<parent link="base_link" />
+    	<child link="rear_camera_link" />
+    	<origin xyz="-0.10 0 0.35" rpy="0 0 0" />
 	</joint>
    </robot>

Commit message: nav now drives straight

File: urdf/robbie.urdf.xacro (robot description, xacro)
@@ -49,5 +49,5 @@
     </visual>
    <collision>
-        <origin xyz="0 0 0" rpy="${M_PI/2} 0 ${M_PI/2}" />
+        <origin xyz="0 0 0" rpy="${M_PI/2} 0 -${M_PI/2}" />
         <geometry>
           <mesh filename="package://omni_bot2/mesh/d435.stl" scale="${M_SCALE} ${M_SCALE} ${M_SCALE}"/>
@@ -88,5 +88,5 @@
     	<parent link="base_link" />
     	<child link="rear_camera_link" />
-    	<origin xyz="-0.10 0 0.35" rpy="0 0 0" />
+    	<origin xyz="-0.10 0 0.35" rpy="0 0 -3.14" />
 	</joint>
    </robot>

Commit message: add arm driver and voice server

File: urdf/robbie.urdf.xacro (robot description, xacro)
@@ -46,8 +46,8 @@
       </geometry>
          <xacro:grey1/>
-      <origin rpy="${M_PI/2} 0 -${M_PI/2}" xyz="0 -0 0"/>
+      <origin rpy="1.57 0 1.57" xyz="0 -0 0"/>
     </visual>
    <collision>
-        <origin xyz="0 0 0" rpy="${M_PI/2} 0 -${M_PI/2}" />
+        <origin xyz="0 0 0" rpy="1.57 0 1.57" />
         <geometry>
           <mesh filename="package://omni_bot2/mesh/d435.stl" scale="${M_SCALE} ${M_SCALE} ${M_SCALE}"/>
@@ -88,5 +88,5 @@
     	<parent link="base_link" />
     	<child link="rear_camera_link" />
-    	<origin xyz="-0.10 0 0.35" rpy="0 0 -3.14" />
+    	<origin xyz="-0.10 0 0.45" rpy="0 0 -0.0" />
 	</joint>
    </robot>

Commit message: new docking system

File: urdf/robbie.urdf.xacro (robot description, xacro)
@@ -7,5 +7,5 @@
   <xacro:include filename="$(find omni_bot2)/urdf/hardware.xacro" />
   <xacro:include filename="$(find omni_bot2)/urdf/materials.xacro" />
-<xacro:my_box name="base_footprint" lwh="0.1 0.1 0.005" xyz="0 0 0" rpy="0 0 0" mass="0.1" material="Gazebo/FlatBlack">
+<xacro:my_box name="base_footprint" lwh="0.4 0.4 0.005" xyz="0 0 0" rpy="0 0 0" mass="0.1" material="Gazebo/FlatBlack">
 	        <xacro:grey2 />
         </xacro:my_box>
@@ -55,5 +55,5 @@
       </collision>
   </link>
-  <link name="front_camera_link" >
+  <link name="oak" >
    <visual>
       <geometry>
@@ -80,7 +80,7 @@
     	<origin xyz="0.15 0 0.32" rpy="0 0 0" />
 	</joint>
-<joint name="front_camera_link" type="fixed">
+<joint name="oak" type="fixed">
     	<parent link="base_link" />
-    	<child link="front_camera_link" />
+    	<child link="oak" />
     	<origin xyz="0.0 0 0.35" rpy="0 0 0" />
 	</joint>
@@ -88,5 +88,5 @@
     	<parent link="base_link" />
     	<child link="rear_camera_link" />
-    	<origin xyz="-0.10 0 0.45" rpy="0 0 -0.0" />
+    	<origin xyz="-0.10 0 0.45" rpy="0 0 3.14" />
 	</joint>
    </robot>
