Commit message: move to RPI5 and ESP32 controller

File: urdf/hardware.xacro (robot description, xacro)
@@ -92,5 +92,5 @@
 				<origin xyz="${xyz}" rpy="${rpy}" />
 				<geometry>
-					<mesh filename="package://omni_bot/mesh/ax12.stl" scale="${M_SCALE} ${M_SCALE} ${M_SCALE}"/>
+					<mesh filename="package://2/mesh/ax12.stl" scale="${M_SCALE} ${M_SCALE} ${M_SCALE}"/>
 				</geometry>
 				<xacro:ax12_color />
@@ -100,5 +100,5 @@
 				<geometry>
 					<!--<box size="0.032 0.038 0.05" />-->
-					<mesh filename="package://omni_bot/mesh/ax12.stl" scale="${M_SCALE} ${M_SCALE} ${M_SCALE}"/>
+					<mesh filename="package://omni_bot2/mesh/ax12.stl" scale="${M_SCALE} ${M_SCALE} ${M_SCALE}"/>
 				</geometry>
              </collision>
@@ -112,12 +112,12 @@
 				<origin xyz="${xyz}" rpy="${rpy}" />
 				<geometry>
-          			<mesh filename="package://omni_bot/mesh/F2.${MESH_EXT}" scale="${M_SCALE} ${M_SCALE} ${M_SCALE}"/>
-				</geometry>
-				<xacro:bracket_color />
-             </visual>
-             <collision>
-				<origin xyz="${xyz}" rpy="${rpy}" />
-					<geometry>
-          				<mesh filename="package://omni_bot/mesh/F2.${MESH_EXT}" scale="${M_SCALE} ${M_SCALE} ${M_SCALE}"/>
+          			<mesh filename="package://omni_bot2/mesh/F2.${MESH_EXT}" scale="${M_SCALE} ${M_SCALE} ${M_SCALE}"/>
+				</geometry>
+				<xacro:bracket_color />
+             </visual>
+             <collision>
+				<origin xyz="${xyz}" rpy="${rpy}" />
+					<geometry>
+          				<mesh filename="package://omni_bot2/mesh/F2.${MESH_EXT}" scale="${M_SCALE} ${M_SCALE} ${M_SCALE}"/>
 					</geometry>
              </collision>
@@ -131,5 +131,5 @@
 				<origin xyz="${xyz}" rpy="${rpy}" />
 				<geometry>
-          			<mesh filename="package://omni_bot/mesh/F3.${MESH_EXT}" scale="${M_SCALE} ${M_SCALE} ${M_SCALE}"/>
+          			<mesh filename="package://omni_bot2/mesh/F3.${MESH_EXT}" scale="${M_SCALE} ${M_SCALE} ${M_SCALE}"/>
 				</geometry><material name="grey1">
 			<color rgba="0.75 0.75 0.75 1.0"/>
@@ -140,5 +140,5 @@
 				<origin xyz="${xyz}" rpy="${rpy}" />
 					<geometry>
-          				<mesh filename="package://omni_bot/mesh/F3.${MESH_EXT}" scale="${M_SCALE} ${M_SCALE} ${M_SCALE}"/>
+          				<mesh filename="package://omni_bot2/mesh/F3.${MESH_EXT}" scale="${M_SCALE} ${M_SCALE} ${M_SCALE}"/>
 					</geometry>
              </collision>

Commit message: change cpu to I7

File: urdf/hardware.xacro (robot description, xacro)
@@ -92,5 +92,5 @@
 				<origin xyz="${xyz}" rpy="${rpy}" />
 				<geometry>
-					<mesh filename="package://2/mesh/ax12.stl" scale="${M_SCALE} ${M_SCALE} ${M_SCALE}"/>
+					<mesh filename="package://omni_bot2/mesh/ax12.stl" scale="${M_SCALE} ${M_SCALE} ${M_SCALE}"/>
 				</geometry>
 				<xacro:ax12_color />
